File: KiCAD/blahajergo.kicad_pcb (KiCad board)
At the start: 2 copper layers, 328.5 x 118.5 mm, 134 parts, among them J1 OLED_128x32, J2 Conn_01x02_Socket, J3 Conn_01x02_Socket, J4 OLED_128x32, SW1 SW_Push, SW2 SW_SPDT, SW3 SW_Push, SW4 SW_SPDT, U1 Nice_Nano_V2, U2 Nice_Nano_V2

Commit message: add mousebites
Parts:
- added G***: LOGO, LOGO, F.Cu at (101.8, 152.5)
- added G***: LOGO, LOGO, F.Cu at (95.8, 152.5)
- added G***: LOGO, LOGO, F.Cu at (327.5, 153.3)
- added G***: LOGO, LOGO, F.Cu at (333.6, 153.2)
- added G***: LOGO, LOGO, B.Cu at (277.0, 165.2)
- added G***: LOGO, LOGO, B.Cu at (152.7, 164.4)
- added mouse-bite-2mm-slot: VAL**, Mousebites:mouse-bite-2mm-slot, F.Cu at (214.7, 133.2)
- added mouse-bite-2mm-slot: VAL**, Mousebites:mouse-bite-2mm-slot, F.Cu at (214.7, 149.2)
- added mouse-bite-2mm-slot: VAL**, Mousebites:mouse-bite-2mm-slot, F.Cu at (214.7, 117.2)
- moved D10 208.4 mm to (262.8, 124.6)
- moved D11 208.4 mm to (262.8, 141.6)
- moved D12 208.4 mm to (262.8, 158.6)
- moved D13 208.4 mm to (287.5, 183.2)
- moved D14 208.4 mm to (280.8, 105.6)
- moved D15 208.4 mm to (280.8, 122.6)
- moved D16 208.4 mm to (280.8, 139.6)
- moved D17 208.4 mm to (280.8, 156.6)
- moved D18 208.4 mm to (307.7, 184.4)
- moved D19 208.4 mm to (298.8, 109.6)
- moved D20 208.4 mm to (298.8, 126.6)
- moved D21 208.4 mm to (298.8, 143.6)
- moved D22 208.4 mm to (298.8, 160.6)
- moved D24 208.4 mm to (316.8, 113.6)
- moved D25 208.4 mm to (316.8, 130.6)
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Other:
- board size 328.5 x 118.5 mm -> 307.4 x 117.3 mm
