File: KiCAD/blahajergo.kicad_pcb (KiCad board)
At the start: 2 copper layers, 307.4 x 117.3 mm, 143 parts, among them J1 OLED_128x32, J2 Conn_01x02_Socket, J3 Conn_01x02_Socket, J4 OLED_128x32, SW1 SW_Push, SW2 SW_SPDT, SW3 SW_Push, SW4 SW_SPDT, U1 Nice_Nano_V2, U2 Nice_Nano_V2

Commit message: REDO: Fix MCU orientation, add support for both choc v1 + v2, new graphics, and new reset switch
Parts:
- removed D1, D10, D11, D12, D13, D14, D15, D16, D17, D18, D19, D2, D20, D21, D22, D23, D24, D25, D26, D27, D28, D3, D4, D5, D6, D7, D8, D9: Diode, chinh4thepro:ComboDiode
- removed the G*** at (101.8, 152.5)
- removed the G*** at (95.8, 152.5)
- removed the G*** at (327.5, 153.3)
- removed the G*** at (333.6, 153.2)
- removed the G*** at (277.0, 165.2)
- removed the G*** at (152.7, 164.4)
- removed J1: OLED_128x32, ScottoKeebs_Components:OLED_128x32
- removed J2: Conn_01x02_Socket, Connector_JST:JST_PH_S2B-PH-K_1x02_P2.00mm_Horizontal
- removed S1, S10, S11, S12, S13, S14, S15, S16, S17, S18, S19, S2, S20, S21, S22, S23, S24, S25, S26, S27, S28, S3, S4, S5, S6, S7, S8, S9: Keyswitch, ScottoKeebs_Hotswap:Hotswap_Choc_V1
- removed SW1: SW_Push, chinh4thepro:SW_TACT_ALPS_SKQGABE010
- removed SW2: SW_SPDT, chinh4thepro:SPDT_C128955
- removed U1: Nice_Nano_V2, ScottoKeebs_MCU:Nice_Nano_V2
- removed _1 (x2), _2 (x2), _3 (x2), _4 (x2), _5 (x2): , MountingHole_2.2mm_M2_Pad_Via
- removed the _6 at (340.1, 160.0)
- removed the _6 at (89.3, 160.0)
- removed mouse-bite-2mm-slot (x3): VAL**, Mousebites:mouse-bite-2mm-slot
- added ?: , , F.Cu at (216.8, 153.3)
- added G***: LOGO, LOGO, F.Cu at (159.1, 138.3)
- added G***: LOGO, LOGO, B.Cu at (210.8, 117.3)
- added _6: , chinh4thepro:MountingHole_2.2mm_M2_Pad_Via, F.Cu at (261.0, 137.7)
- added _6: , chinh4thepro:MountingHole_2.2mm_M2_Pad_Via, F.Cu at (169.4, 91.5)
- added _6: , chinh4thepro:MountingHole_2.2mm_M2_Pad_Via, F.Cu at (157.3, 158.7)
- added _6: , chinh4thepro:MountingHole_2.2mm_M2_Pad_Via, F.Cu at (261.2, 103.8)
- S29, S30, S31, S32, S33, S34, S35, S36, S37, S38, S39, S40, S41, S42, S43, S44, S45, S46, S47, S48, S49, S50, S51, S52, S53, S54, S55, S56: footprint ScottoKeebs_Hotswap:Hotswap_Choc_V1 -> ScottoKeebs_Hotswap:Hotswap_Choc_V1V2
- SW3: footprint chinh4thepro:SW_TACT_ALPS_SKQGABE010 -> Button_Switch_SMD:Panasonic_EVQPUL_EVQPUC
- U2: footprint ScottoKeebs_MCU:Nice_Nano_V2 -> ScottoKeebs_MCU:Nice_Nano_V2_Flipped
- moved D44 70.7 mm to (218.1, 126.2)
- moved D52 70.7 mm to (182.1, 100.2)
- moved D53 70.7 mm to (182.1, 117.2)
- moved D54 70.7 mm to (182.1, 134.2)
- moved D55 70.7 mm to (182.1, 151.2)
- moved D29 70.7 mm to (272.1, 100.2)
- moved D30 70.7 mm to (272.1, 117.2)
- moved D31 70.7 mm to (272.1, 134.2)
- moved D32 70.7 mm to (272.1, 151.2)
- moved D33 70.7 mm to (254.1, 100.2)
- moved D34 70.7 mm to (254.1, 117.2)
- moved D35 70.7 mm to (254.1, 134.2)
- moved D36 70.7 mm to (254.1, 151.2)
- moved D37 70.7 mm to (236.1, 94.2)
- moved D38 70.7 mm to (236.1, 111.2)
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Routing:
- net L_COL4: track 265.2 -> 0.00 mm
- net L_COL5: track 238.1 -> 0.00 mm
- net L_COL3: track 211.8 -> 0.00 mm
- net L_ROW4: track 193.4 -> 0.00 mm
- net L_COL6: track 188.9 -> 0.00 mm
- net L_ROW5: track 180.8 -> 0.00 mm
- net L_COL1: track 178.6 -> 0.00 mm
- net L_ROW3: track 174.7 -> 0.00 mm
- net L_ROW2: track 162.4 -> 0.00 mm
- net L_COL2: track 160.1 -> 0.00 mm
- net L_ROW1: track 158.7 -> 0.00 mm
- net GND: track 267.6 -> 155.5 mm
- net L_BAT_RAW: track 60.4 -> 0.00 mm
- net R_ROW2: track 206.6 -> 152.3 mm
- net L_RST: track 49.3 -> 0.00 mm
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Other:
- board size 307.4 x 117.3 mm -> 151.3 x 126.2 mm
- board text added: "3.3v"
- board text added: "B+"
- board text added: "D0"
- board text added: "D1"
- board text added: "D10"
- board text added: "D14"
- board text added: "D15"
- board text added: "D16"
- board text added: "D18"
- board text added: "D19"
- board text added: "D2"
- board text added: "D20"
- board text added: "D21"
- board text added: "D3"
- board text added: "D4"
- board text added: "D5"
- board text added: "D6"
- board text added: "D7"
- board text added: "D8"
- board text added: "D9"
- board text added: "GND"
- board text added: "RST"

Commit message: update readme
Parts:
- removed ?: , 
- added _6: , chinh4thepro:MountingHole_2.2mm_M2_Pad_Via, F.Cu at (220.0, 151.0)
Changed lines of the file:
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@@
 		)
 		(fp_line
-			(start 7.281012 -5.608985)
+			(start 7.281012 -5.608984)
 			(end 7.366007 -5.181999)
 			(stroke
@@
 		(fp_line
 			(start 7.092007 -5.892008)
-			(end 7.281012 -5.608985)
+			(end 7.281012 -5.608984)
 			(stroke
 				(width 0.12)
@@
 		(fp_line
 			(start -1.523003 -3.447992)
-			(end -2.452008 -4.376998)
+			(end -2.452008 -4.376997)
 			(stroke
 				(width 0.05)
@@
 		)
 		(fp_line
-			(start -2.452008 -4.376998)
+			(start -2.452008 -4.376997)
 			(end -2.452014 -7.522994)
 			(stroke
@@
 		(fp_line
 			(start 3.210998 -1.311992)
-			(end 2.903002 -1.502992)
+			(end 2.903001 -1.502992)
 			(stroke
 				(width 0.05)
@@
 		)
 		(fp_line
-			(start 2.903002 -1.502992)
+			(start 2.903001 -1.502992)
 			(end 2.687009 -1.793999)
 			(stroke
@@
 		(fp_line
 			(start -0.749999 -0.000001)
-			(end -0.350002 -0.000001)
+			(end -0.350002 0)
 			(stroke
 				(width 0.1)
@@
 		)
 		(fp_line
-			(start -0.350002 -0.000001)
+			(start -0.350002 0)
 			(end -0.350001 -0.550001)
 			(stroke
@@
 		)
 		(fp_line
-			(start -0.350002 -0.000001)
+			(start -0.350002 0)
 			(end -0.35 0.55)
 			(stroke
@@
 		)
 		(fp_line
-			(start -0.350002 -0.000001)
+			(start -0.350002 0)
 			(end 0.25 -0.4)
 			(stroke
@@
 		)
 		(fp_line
-			(start 0.250001 0.000001)
+			(start 0.250001 0.000002)
 			(end 0.749999 0.000001)
 			(stroke
@@
 		(fp_line
 			(start 0.25 0.399999)
-			(end -0.350002 -0.000001)
+			(end -0.350002 0)
 			(stroke
 				(width 0.1)
@@
 		(fp_line
 			(start -0.749999 -0.000001)
-			(end -0.350002 -0.000001)
+			(end -0.350002 0)
 			(stroke
 				(width 0.1)
@@
 		)
 		(fp_line
-			(start -0.350002 -0.000001)
+			(start -0.350002 0)
 			(end -0.350001 -0.550001)
 			(stroke
@@
 		)
 		(fp_line
-			(start -0.350002 -0.000001)
+			(start -0.350002 0)
 			(end -0.35 0.55)
 			(stroke
@@
 		)
 		(fp_line
-			(start -0.350002 -0.000001)
+			(start -0.350002 0)
 			(end 0.25 -0.4)
 			(stroke
@@
 		)
 		(fp_line
-			(start 0.250001 0.000001)
+			(start 0.250001 0.000002)
 			(end 0.749999 0.000001)
 			(stroke
@@
 		(fp_line
 			(start 0.25 0.399999)
-			(end -0.350002 -0.000001)
+			(end -0.350002 0)
 			(stroke
 				(width 0.1)
@@
 		)
 	)
+	(footprint "chinh4thepro:MountingHole_2.2mm_M2_Pad_Via"
+		(layer "F.Cu")
+		(at 220 151)
+		(property "Reference" "_6"
+			(at 0 -3.2 0)
+			(layer "F.SilkS")
+			(hide yes)
+			(effects
+				(font
+					(size 1 1)
+					(thickness 0.15)
+				)
+			)
+		)
+		(property "Value" ""
+			(at 0 0 0)
+			(layer "F.SilkS")
+			(hide yes)
+			(effects
+				(font
+					(size 1.27 1.27)
+					(thickness 0.15)
+				)
+			)
+		)
+		(property "Footprint" "chinh4thepro:MountingHole_2.2mm_M2_Pad_Via"
+			(at 0 0 0)
+			(unlocked yes)
+			(layer "F.Fab")
+			(hide yes)
+			(effects
+				(font
+					(size 1.27 1.27)
+				)
+			)
+		)
+		(property "Datasheet" ""
+			(at 0 0 0)
+			(unlocked yes)
+			(layer "F.Fab")
+			(hide yes)
+			(effects
+				(font
+					(size 1.27 1.27)
+				)
+			)
+		)
+		(property "Description" ""
+			(at 0 0 0)
+			(unlocked yes)
+			(layer "F.Fab")
+			(hide yes)
+			(effects
+				(font
+					(size 1.27 1.27)
+				)
+			)
+		)
+		(fp_circle
+			(center 0 0)
+			(end 2.45 0)
+			(stroke
+				(width 0.05)
+				(type solid)
+			)
+			(fill none)
+			(layer "F.CrtYd")
+		)
+		(pad "1" thru_hole circle
+			(at -1.65 0)
+			(size 0.7 0.7)
+			(drill 0.4)
+			(layers "*.Cu" "*.Mask")
+			(remove_unused_layers no)
+		)
+		(pad "1" thru_hole circle
+			(at -1.166726 -1.166726)
+			(size 0.7 0.7)
+			(drill 0.4)
+			(layers "*.Cu" "*.Mask")
+			(remove_unused_layers no)
+		)
+		(pad "1" thru_hole circle
+			(at -1.166726 1.166726)
+			(size 0.7 0.7)
+			(drill 0.4)
+			(layers "*.Cu" "*.Mask")
+			(remove_unused_layers no)
+		)
+		(pad "1" thru_hole circle
+			(at 0 -1.65)
+			(size 0.7 0.7)
+			(drill 0.4)
+			(layers "*.Cu" "*.Mask")
+			(remove_unused_layers no)
+		)
+		(pad "1" thru_hole circle
+			(at 0 0)
+			(size 4.4 4.4)
+			(drill 2.2)
+			(layers "*.Cu" "*.Mask")
+			(remove_unused_layers no)
+		)
+		(pad "1" thru_hole circle
+			(at 0 1.65)
+			(size 0.7 0.7)
+			(drill 0.4)
+			(layers "*.Cu" "*.Mask")
+			(remove_unused_layers no)
+		)
+		(pad "1" thru_hole circle
+			(at 1.166726 -1.166726)
+			(size 0.7 0.7)
+			(drill 0.4)
+			(layers "*.Cu" "*.Mask")
+			(remove_unused_layers no)
+		)
+		(pad "1" thru_hole circle
+			(at 1.166726 1.166726)
+			(size 0.7 0.7)
+			(drill 0.4)
+			(layers "*.Cu" "*.Mask")
+			(remove_unused_layers no)
+		)
+		(pad "1" thru_hole circle
+			(at 1.65 0)
+			(size 0.7 0.7)
+			(drill 0.4)
+			(layers "*.Cu" "*.Mask")
+			(remove_unused_layers no)
+		)
+	)
 	(footprint "chinh4thepro:ComboDiode"
 		(layer "F.Cu")
@@
 		(fp_line
 			(start 6.85 -6.181001)
-			(end 7.168001 -5.968)
+			(end 7.168001 -5.968001)
 			(stroke
 				(width 0.05)
@@
 		)
 		(fp_line
-			(start 7.168001 -5.968)
+			(start 7.168001 -5.968001)
 			(end 7.381001 -5.65)
 			(stroke
@@
 		(fp_line
 			(start 3.216 -6.166001)
-			(end 3.675 -6.075001)
+			(end 3.674999 -6.075001)
 			(stroke
 				(width 0.1)
@@
 		)
 		(fp_line
-			(start 3.675 -6.075001)
+			(start 3.674999 -6.075001)
 			(end 6.474998 -6.074998)
 			(stroke
@@
 		(tags "SMD SMT SPST EVQPUL EVQPUC")
 		(property "Reference" "SW3"
-			(at -0.000002 -4.499998 270)
+			(at -0.000002 -4.499998 -90)
 			(layer "F.SilkS")
 			(hide yes)
@@
 		)
 		(property "Value" "SW_Push"
-			(at 0 3.5 270)
+			(at 0 3.5 -90)
 			(layer "F.Fab")
 			(hide yes)
@@
 		(at 149.994999 123.875003 90)
 		(property "Reference" "J4"
-			(at 7.750002 10 270)
+			(at 7.750002 10 -90)
 			(layer "F.SilkS")
 			(hide yes)
@@
 		)
 		(property "Value" "OLED_128x32"
-			(at 5.749999 5.750002 270)
+			(at 5.749999 5.750002 -90)
 			(layer "F.Fab")
 			(hide yes)
@@
 		)
 	)
-	(footprint ""
-		(layer "F.Cu")
-		(at 216.85 153.325)
-		(property "Reference" ""
-			(at 0 0 0)
-			(unlocked yes)
-			(layer "F.SilkS")
-			(hide yes)
-			(effects
-				(font
-					(size 1.27 1.27)
-				)
-			)
-		)
-		(property "Value" ""
-			(at 0 0 0)
-			(unlocked yes)
-			(layer "F.Fab")
-			(hide yes)
-			(effects
-				(font
-					(size 1.27 1.27)
-				)
-			)
-		)
-		(property "Footprint" ""
-			(at 0 0 0)
-			(unlocked yes)
-			(layer "F.Fab")
-			(hide yes)
-			(effects
-				(font
-					(size 1.27 1.27)
-				)
-			)
-		)
-		(property "Datasheet" ""
-			(at 0 0 0)
-			(unlocked yes)
-			(layer "F.Fab")
-			(hide yes)
-			(effects
-				(font
-					(size 1.27 1.27)
-				)
-			)
-		)
-		(property "Description" ""
-			(at 0 0 0)
-			(unlocked yes)
-			(layer "F.Fab")
-			(hide yes)
-			(effects
-				(font
-					(size 1.27 1.27)
-				)
-			)
-		)
-		(pad "1" thru_hole circle
-			(at 0 0)
-			(size 4.4 4.4)
-			(drill 2.2)
-			(layers "*.Cu" "*.Mask")
-			(remove_unused_layers no)
-		)
-	)
 	(footprint "ScottoKeebs_Hotswap:Hotswap_Choc_V1V2"
 		(layer "F.Cu")
@@
 		)
 		(fp_line
-			(start -1.479 -3.554001)
-			(end -2.499998 -4.575)
+			(start -1.479001 -3.554001)
+			(end -2.499998 -4.575001)
 			(stroke
 				(width 0.12)
@@
 		(fp_line
 			(start 1.671 -8.265999)
-			(end 2.012999 -8.037)
+			(end 2.012998 -8.037)
 			(stroke
 				(width 0.12)
@@
 		(fp_line
 			(start 1.168001 -3.553999)
-			(end -1.479 -3.554001)
+			(end -1.479001 -3.554001)
 			(stroke
 				(width 0.12)
@@
 		)
 		(fp_line
-			(start 2.012999 -8.037)
+			(start 2.012998 -8.037)
 			(end 2.546001 -7.503999)
 			(stroke
@@
 		(fp_line
 			(start 2.633001 -6.844)
-			(end 2.877001 -6.477)
+			(end 2.877002 -6.477)
 			(stroke
 				(width 0.12)
@@
 		)
 		(fp_line
-			(start 2.877001 -6.477)
+			(start 2.877002 -6.477)
 			(end 3.243999 -6.233001)
 			(stroke
@@
 		(fp_line
 			(start 7.092 -5.891999)
-			(end 7.281001 -5.608999)
+			(end 7.281 -5.608999)
 			(stroke
 				(width 0.12)
@@
 		)
 		(fp_line
-			(start 7.281001 -5.608999)
+			(start 7.281 -5.608999)
 			(end 7.366001 -5.182)
 			(stroke
