File: KiCAD/blahajergo.kicad_pcb (KiCad board)
At the start: 2 copper layers, 306.1 x 134.2 mm, 144 parts, among them J1 OLED_128x32, J2 Conn_01x02_Socket, J3 Conn_01x02_Socket, J4 OLED_128x32, SW1 SW_Push, SW2 SW_SPDT, SW3 SW_Push, SW4 SW_SPDT, U1 Nice_Nano_V2, U2 Nice_Nano_V2

Commit message: flip jst connector terminals
Parts:
- J2, J3: moved to B.Cu
- moved J2 1.98 mm to (353.3, 134.7), turned to 180 degrees
- moved J3 1.95 mm to (77.7, 134.7), turned to 180 degrees
Routing:
- net GND: track 241.5 -> 237.6 mm
- net R_BAT_IN: track 19.7 -> 20.2 mm
