File: KiCAD/blahajergo.kicad_sch (KiCad schematic)
At the start: 122 parts, among them J1 OLED_128x32, J2 Conn_01x02_Socket, J3 Conn_01x02_Socket, J4 OLED_128x32, SW1 SW_Push, SW2 SW_SPDT, SW3 SW_Push, SW4 SW_SPDT, U1 Nice_Nano_V2, U2 Nice_Nano_V2

Commit message: REDO: Fix MCU orientation, add support for both choc v1 + v2, new graphics, and new reset switch
Parts:
- S1, S10, S11, S12, S13, S14, S15, S16, S17, S18, S19, S2, S20, S21, S22, S23, S24, S25, S26, S27, S28, S29, S3, S30, S31, S32, S33, S34, S35, S36, S37, S38, S39, S4, S40, S41, S42, S43, S44, S45, S46, S47, S48, S49, S5, S50, S51, S52, S53, S54, S55, S56, S6, S7, S8, S9: footprint ScottoKeebs_Hotswap:Hotswap_Choc_V1 -> ScottoKeebs_Hotswap:Hotswap_Choc_V1V2
- SW1, SW3: footprint chinh4thepro:SW_TACT_ALPS_SKQGABE010 -> Button_Switch_SMD:Panasonic_EVQPUL_EVQPUC
- U1, U2: footprint ScottoKeebs_MCU:Nice_Nano_V2 -> ScottoKeebs_MCU:Nice_Nano_V2_Flipped

Commit message: finally finish pcb redo
Connections:
- net L_COL1: now also U1.7 (D4); no longer U1.1 (D1)
- net L_COL3: now also U1.1 (D1); no longer U1.12 (D9)
- net L_COL4: now also U1.13 (D10); no longer U1.15 (D14)
- net L_COL6: now also U1.15 (D14); no longer U1.13 (D10)
- net L_ROW1: now also U1.20 (D21); no longer U1.7 (D4)
- net L_ROW2: now also U1.19 (D20); no longer U1.8 (D5)
- net L_ROW3: now also U1.18 (D19); no longer U1.9 (D6)
- net L_ROW4: now also U1.17 (D18); no longer U1.10 (D7)
- net L_ROW5: now also U1.16 (D15); no longer U1.11 (D8)
